File: DMH-Kosmo-10cm-PCB/DMH-Kosmo-10cm-PCB.kicad_pcb (KiCad board)
At the start: 2 copper layers, 96 x 175 mm, 0 parts

Commit message: Added template meta data and JLC SN placeholder
Other:
- board text added: "JLCJLCJLCJLC"
Changed lines of the file:
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@@
 		(layer "User.9")
 	)
+	(gr_text "JLCJLCJLCJLC"
+		(at 100 45 0)
+		(layer "B.SilkS")
+		(effects
+			(font
+				(size 1 1)
+				(thickness 0.15)
+			)
+			(justify mirror)
+		)
+	)
 )

Commit message: Updated 5cm and 10 templates
Other:
- board text added: "Mk1.0 - Month Year"
- board text removed: "JLCJLCJLCJLC"
Changed lines of the file:
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@@
 	(net 0 "")
+	(gr_rect
+		(start 95 212.75)
+		(end 105 214.75)
+		(stroke
+			(width 0.1)
+			(type solid)
+		)
+		(fill solid)
+		(layer "B.SilkS")
+	)
 	(gr_rect
 		(start 52 42.5)
@@
 		(layer "User.9")
 	)
-	(gr_text "JLCJLCJLCJLC"
-		(at 100 45 0)
+	(gr_text "Mk1.0 - Month Year"
+		(at 100 216.25 0)
 		(layer "B.SilkS")
 		(effects
 			(font
 				(size 1 1)
-				(thickness 0.15)
+				(thickness 0.25)
+				(bold yes)
 			)
 			(justify mirror)
