File: DMH-Kosmo-5cm-PCB/Inputs_and_Outputs.kicad_sch (KiCad schematic)
At the start: 0 parts

Commit message: Added initial jacks and connectors to PCBs
Parts:
- added J1, J2, J3, J4: TS_Jack_6.35mm_Sw, SynthStuff:CUI_MJ-63052A, symbol SynthStuff:TS_Jack_6.35mm_Sw
- added J200: IDC_02x05, SynthStuff:IDC-Header_2x05_P2.54mm_Vertical_BackBone, symbol SynthStuff:BackBone_Connector_10Pin
- added J50, J60: Conn_01x06, Connector_PinSocket_2.54mm:PinSocket_1x06_P2.54mm_Vertical, symbol Connector_Generic:Conn_01x06
