File: DMH-Kosmo-15cm-PCB/Power.kicad_sch (KiCad schematic)
At the start: 13 parts, among them J0 Conn_01x01, J100 IDC_02x05, J101 IDC_02x08

Commit message: Updated power components
- Changed Schottky Diodes from SB140 to 1N5819
- Reduced electrolytic caps from 47uF to 22uF
Parts:
- C1, C2, C5: value 47uF -> 22uF
- D1, D2, D3, D4, D5: value SB140 -> 1N5819; symbol Diode:SB140 -> Diode:1N5819
Changed lines of the file:
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@@
 	)
 	(symbol
-		(lib_id "Diode:SB140")
+		(lib_id "Diode:1N5819")
 		(at 109.22 175.26 0)
 		(unit 1)
@@
 			)
 		)
-		(property "Value" "SB140"
+		(property "Value" "1N5819"
 			(at 108.9025 171.45 0)
 			(show_name no)
@@
 			)
 		)
-		(property "Datasheet" "http://www.diodes.com/_files/datasheets/ds23022.pdf"
+		(property "Datasheet" "http://www.vishay.com/docs/88525/1n5817.pdf"
 			(at 109.22 175.26 0)
 			(hide yes)
@@
 			)
 		)
-		(property "Value" "47uF"
+		(property "Value" "22uF"
 			(at 29.21 133.7309 0)
 			(show_name no)
@@
 			)
 		)
-		(property "Value" "47uF"
+		(property "Value" "22uF"
 			(at 29.21 38.4809 0)
 			(show_name no)
@@
 	)
 	(symbol
-		(lib_id "Diode:SB140")
+		(lib_id "Diode:1N5819")
 		(at 53.34 175.26 0)
 		(unit 1)
@@
 			)
 		)
-		(property "Value" "SB140"
+		(property "Value" "1N5819"
 			(at 53.0225 171.45 0)
 			(show_name no)
@@
 			)
 		)
-		(property "Datasheet" "http://www.diodes.com/_files/datasheets/ds23022.pdf"
+		(property "Datasheet" "http://www.vishay.com/docs/88525/1n5817.pdf"
 			(at 53.34 175.26 0)
 			(hide yes)
@@
 	)
 	(symbol
-		(lib_id "Diode:SB140")
+		(lib_id "Diode:1N5819")
 		(at 53.34 185.42 180)
 		(unit 1)
@@
 			)
 		)
-		(property "Value" "SB140"
+		(property "Value" "1N5819"
 			(at 53.6575 181.61 0)
 			(show_name no)
@@
 			)
 		)
-		(property "Datasheet" "http://www.diodes.com/_files/datasheets/ds23022.pdf"
+		(property "Datasheet" "http://www.vishay.com/docs/88525/1n5817.pdf"
 			(at 53.34 185.42 0)
 			(hide yes)
@@
 	)
 	(symbol
-		(lib_id "Diode:SB140")
+		(lib_id "Diode:1N5819")
 		(at 53.34 195.58 180)
 		(unit 1)
@@
 			)
 		)
-		(property "Value" "SB140"
+		(property "Value" "1N5819"
 			(at 53.6575 191.77 0)
 			(show_name no)
@@
 			)
 		)
-		(property "Datasheet" "http://www.diodes.com/_files/datasheets/ds23022.pdf"
+		(property "Datasheet" "http://www.vishay.com/docs/88525/1n5817.pdf"
 			(at 53.34 195.58 0)
 			(hide yes)
@@
 	)
 	(symbol
-		(lib_id "Diode:SB140")
+		(lib_id "Diode:1N5819")
 		(at 109.22 185.42 180)
 		(unit 1)
@@
 			)
 		)
-		(property "Value" "SB140"
+		(property "Value" "1N5819"
 			(at 109.5375 181.61 0)
 			(show_name no)
@@
 			)
 		)
-		(property "Datasheet" "http://www.diodes.com/_files/datasheets/ds23022.pdf"
+		(property "Datasheet" "http://www.vishay.com/docs/88525/1n5817.pdf"
 			(at 109.22 185.42 0)
 			(hide yes)
@@
 			)
 		)
-		(property "Value" "47uF"
+		(property "Value" "22uF"
 			(at 29.21 108.3309 0)
 			(show_name no)
